Commit message: Update full features done in laser scan detection, image processing, spawn model

File: conveyor/urdf/blue_cube.urdf (robot description, URDF)
Before this commit: robot blue_cube, 1 links, 0 joints
Links:
- link base_link: geometry collision box size=0.08 0.08 0.08; visual box size=0.08 0.08 0.08

File: conveyor/urdf/conveyor.urdf.xacro (robot description, xacro)
@@ -48,5 +48,5 @@
 		<child link="belt$(arg system)_moving"/>
 		<axis xyz="0 1 0"/>
-		<limit lower="0.0" upper="1" effort="1000" velocity="1000"/>
+		<limit lower="0.0" upper="0.1" effort="1000" velocity="1000"/>
 	</joint>
 	<link name="belt$(arg system)_moving">
@@ -59,5 +59,5 @@
 			<origin xyz="0.0 0.0 0.0005" rpy="0.0 0.0 0.0"/>
 			<geometry>
-				<box size="0.3 1.2 0.001"/>
+				<box size="0.3 1.25 0.001"/>
 			</geometry>
 			<material name="black">
@@ -67,5 +67,5 @@
 			<origin xyz="0.0 0.0 0.0005" rpy="0.0 0.0 0.0"/>
 			<geometry>
-				<box size="0.3 1.2 0.001"/>
+				<box size="0.3 1.17 0.001"/>
 			</geometry>
 		</collision>
@@ -80,6 +80,6 @@
 		<plugin name="conveyor_belt_plugin" filename="libROSConveyorBeltPlugin.so">
 			<robot_namespace>/</robot_namespace>
-			<link>belt_moving</link>
-			<power>40</power>
+			<link>belt$(arg system)_moving</link>
+			<power>30</power>
 			<control_topic>conveyor/control$(arg system)</control_topic>
 			<state_topic>conveyor/state$(arg system)</state_topic>

File: conveyor/urdf/green_cube.urdf (robot description, URDF)
Before this commit: robot green_cube, 1 links, 0 joints
Links:
- link base_link: geometry collision box size=0.08 0.08 0.08; visual box size=0.08 0.08 0.08

File: conveyor/urdf/lidar.urdf.xacro (robot description, xacro)
@@ -26,5 +26,5 @@
         </xacro:inertial_box>
     </link>
-    <joint name="laser_frame" type="fixed">
+    <joint name="laser_joint" type="fixed">
         <parent link="laser_link"/>
         <child link="laser_frame"/>

File: conveyor/urdf/red_cube.urdf (robot description, URDF)
Before this commit: robot red_cube, 1 links, 0 joints
Links:
- link base_link: geometry collision box size=0.08 0.08 0.08; visual box size=0.08 0.08 0.08
